Commit message: updated urdf

File: urdf/jaguar.urdf (robot description, URDF)
Before this commit: robot jaguar_robot, 3 links, 2 joints
Links:
- removed link os1_sensor
- added link os1_lidar
Joints:
- removed joint os1_sensor
- added joint os1_lidar_joint: type fixed, parent base_link, child os1_lidar, origin xyz=-0.01936 0 0.64805 rpy=0 0 ${PI}
- joint imu_joint: origin xyz=0 0 0 rpy=0 0 0 -> xyz=0.14653 0 0.34964 rpy=0 0 0

Commit message: added map saving to rosbag at the end

File: urdf/jaguar.urdf (robot description, URDF)
Before this commit: robot jaguar_robot, 3 links, 2 joints
Links:
- added link navsat_link
Joints:
- removed joint os1_lidar
- added joint navsat_joint: type fixed, parent base_link, child navsat_link, origin xyz=0 0 0 rpy=0 0 0
- added joint os1_lidar_joint: type fixed, parent base_link, child os1_lidar, origin xyz=-0.01936 0 0.64805 rpy=0 0 ${PI}
- joint imu_joint: origin xyz=0 0 0 rpy=0 0 0 -> xyz=0.14653 0 0.34964 rpy=0 0 0

Commit message: reflecting ouster pkg updates

File: urdf/jaguar.urdf (robot description, URDF)
Before this commit: robot jaguar_robot, 4 links, 3 joints
Links:
- removed link os1_lidar
- added link os_sensor
Joints:
- removed joint os1_lidar_joint
- added joint os_sensor_joint: type fixed, parent base_link, child os_sensor, origin xyz=-0.01936 0 0.64805 rpy=0 0 0

Commit message: saga config

File: urdf/jaguar.urdf (robot description, URDF)
Before this commit: robot jaguar_robot, 4 links, 3 joints
Links:
- removed link imu_link
- added link xsens
Joints:
- joint imu_joint: child imu_link -> xsens; origin xyz=0.14653 0 0.34964 rpy=0 0 0 -> xyz=0 0 0 rpy=0 0 0
- joint os_sensor_joint: origin xyz=-0.01936 0 0.64805 rpy=0 0 0 -> xyz=0 0 0 rpy=0 0 0

Commit message: updated urdf

File: urdf/jaguar.urdf (robot description, URDF)
Before this commit: robot jaguar_robot, 4 links, 3 joints
Joints:
- joint imu_joint: origin xyz=0 0 0 rpy=0 0 0 -> xyz=0 0.03 1.3 rpy=0 0 0
- joint os_sensor_joint: origin xyz=0 0 0 rpy=0 0 0 -> xyz=0 0.3 1.3 rpy=0 0 0
